Commit message: Launch file and initial links
Added launch file and all links. Not sure how to connect "circularly", will have to figure this out. Need to add realistic speed, torque and max/min rotation.

File: urdf/manipulator.urdf (robot description, URDF)
Before this commit: robot lift-arm, 2 links, 1 joints
Links:
- added link rack_link; visual mesh filename=package://my_arm_description/models/meshes/collada_files/ra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
- added link sec_arm_link; visual mesh filename=package://my_arm_description/models/meshes/collada_files/se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
- added link strut_link; visual mesh filename=package://my_arm_description/models/meshes/collada_files/st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
- added link upper_arm_link; visual mesh filename=package://my_arm_description/models/meshes/collada_files/up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
- link base_link: geometry visual mesh filename=package://my_arm_description/models/meshes/collada_files/ba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
- link main_arm_link: geometry visual mesh filename=package://my_arm_description/models/meshes/collada_files/ma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
Joints:
- added joint rack_joint: type prismatic, parent upper_arm_link, child rack_link, origin xyz=0 0 0.033 rpy=0 0 -1.571, axis 1 0 0, limit lower=-0.1 upper=0.15 effort=0.1 velocity=0.005
- added joint sec_arm_joint: type revolute, parent base_link, child sec_arm_link, origin xyz=0 0.0095 0.044953 rpy=0 0 1.571, axis 1 0 0, limit lower=-0.2 upper=0.2 effort=0.1 velocity=0.005
- added joint strut_joint_lower: type continuous, parent sec_arm_link, child strut_link, origin xyz=0.006 0.09 0 rpy=0 0 0, axis 1 0 0
- added joint upper_arm_joint: type revolute, parent main_arm_link, child upper_arm_link, origin xyz=0.0095 0 0.18 rpy=0 0 0, axis 1 0 0, limit lower=-0.2 upper=0.2 effort=0.1 velocity=0.005
- joint main_arm_joint: child roll_M1_link -> main_arm_link; origin xyz=0.0023 0 -0.0005 rpy=0 0 0 -> xyz=0 -0.0095 0.044953 rpy=0 0 1.571

Commit message: added xacro macro
and collision data

File: urdf/manipulator.urdf (robot description, URDF)
Before this commit: robot lift-arm, 6 links, 5 joints
Links:
- link base_link: geometry collision mesh filename=package://lift-arm-description/models/meshes/collada_files/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; visual mesh filename=package://lift-arm-description/models/meshes/collada_files/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
- link main_arm_link: geometry collision mesh filename=package://lift-arm-description/models/meshes/collada_files/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; visual mesh filename=package://lift-arm-description/models/meshes/collada_files/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
- link rack_link: geometry collision mesh filename=package://lift-arm-description/models/meshes/collada_files/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; visual mesh filename=package://lift-arm-description/models/meshes/collada_files/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
- link sec_arm_link: geometry collision mesh filename=package://lift-arm-description/models/meshes/collada_files/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; visual mesh filename=package://lift-arm-description/models/meshes/collada_files/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
- link strut_link: geometry collision mesh filename=package://lift-arm-description/models/meshes/collada_files/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; visual mesh filename=package://lift-arm-description/models/meshes/collada_files/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
- link upper_arm_link: geometry collision mesh filename=package://lift-arm-description/models/meshes/collada_files/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; visual mesh filename=package://lift-arm-description/models/meshes/collada_files/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
Joints:
- joint main_arm_joint: limit lower=-0.2 upper=0.2 effort=0.1 velocity=0.005 -> lower=-1.920 upper=1.134 effort=0.1 velocity=0.005
- joint sec_arm_joint: limit lower=-0.2 upper=0.2 effort=0.1 velocity=0.005 -> lower=-0.436 upper=2.531 effort=0.1 velocity=0.005
- joint upper_arm_joint: limit lower=-0.2 upper=0.2 effort=0.1 velocity=0.005 -> lower=-0.873 upper=1.484 effort=0.1 velocity=0.005
