Commit message: added physics
and some new meshes

File: robot/manipulator_macro.xacro (robot description, xacro)
@@ -3,113 +3,173 @@
 	<xacro:macro name="lift-arm" params="prefix">
 		<link name="${prefix}base_link">
-		  <visual>
-		    <origin rpy="0 0 3.142" xyz="0 0 0"/>
-		    <geometry>
-		      <mesh filename="package://lift-arm-description/models/meshes/collada_files/base.dae"/>
-		    </geometry>
-		  </visual>
-		  <collision>
-		  	<origin rpy="0 0 3.142" xyz="0 0 0"/>
-		    <geometry>
-		      <mesh filename="package://lift-arm-description/models/meshes/collada_files/base.dae"/>
-		  	</geometry>
-		  </collision>
+			<inertial>
+				<origin rpy="0 0 0" xyz="0 -0.04 0"/>
+				<mass value="0.873"/>
+				<inertia
+					ixx="0.001751"
+					ixy="0.000012"	iyy="0.000963"
+					ixz="0"			iyz="0.000002"	izz="0.001730"
+				/>
+			</inertial>
+			<visual>
+				<origin rpy="0 0 3.142" xyz="0 0 0"/>
+				<geometry>
+					<mesh filename="package://lift-arm-description/models/meshes/collada_files/base.dae"/>
+				</geometry>
+			</visual>
+			<collision>
+				<origin rpy="0 0 3.142" xyz="0 0 0"/>
+				<geometry>
+					<mesh filename="package://lift-arm-description/models/meshes/collada_files/base.dae"/>
+				</geometry>
+				<contact_coefficients mu="1" kp="100000" kd="100000"/>
+			</collision>
 		</link>
 		<link name="${prefix}main_arm_link">
-		  <visual>
-		    <origin rpy="1.571 -1.571 1.571" xyz="0 0 0"/>
-		    <geometry>
-		      <mesh filename="package://lift-arm-description/models/meshes/collada_files/main_arm.dae"/>
-		    </geometry>
-		  </visual>
-		  <collision>
-		  	<origin rpy="1.571 -1.571 1.571" xyz="0 0 0"/>
-		    <geometry>
-		      <mesh filename="package://lift-arm-description/models/meshes/collada_files/main_arm.dae"/>
-		  	</geometry>
-		  </collision>
+			<inertial>
+				<origin rpy="0 0 0" xyz="0.062 0.007 0.004"/>
+				<mass value="0.108"/>
+				<inertia
+					ixx="0.000028"
+					ixy="-0.000009"	iyy="0.000447"
+					ixz="0.000031"	iyz="-0.000002"	izz="0.000453"
+				/>
+			</inertial>
+			<visual>
+				<origin rpy="1.571 -1.571 1.571" xyz="0 0 0"/>
+				<geometry>
+					<mesh filename="package://lift-arm-description/models/meshes/collada_files/main_arm.dae"/>
+				</geometry>
+			</visual>
+			<collision>
+				<origin rpy="1.571 -1.571 1.571" xyz="0 0 0"/>
+				<geometry>
+					<mesh filename="package://lift-arm-description/models/meshes/collada_files/main_arm.dae"/>
+				</geometry>
+				<contact_coefficients mu="1" kp="100000" kd="100000"/>
+			</collision>
 		</link>
 		<joint name="${prefix}main_arm_joint" type="revolute">
-		  <parent link="${prefix}base_link"/>
-		  <child link="${prefix}main_arm_link"/>
-		  <origin xyz="0 -0.0095 0.044953" rpy="0 0 1.571"/>
-		  <limit lower="-1.920" upper="1.134" effort="2.236" velocity="7.480"/>
-		  <axis xyz="1 0 0"/>
+			<parent link="${prefix}base_link"/>
+			<child link="${prefix}main_arm_link"/>
+			<origin xyz="0 -0.0095 0.044953" rpy="0 0 1.571"/>
+			<limit lower="-1.920" upper="1.134" effort="2.236" velocity="7.480"/>
+			<axis xyz="1 0 0"/>
 		</joint>
 		<link name="${prefix}sec_arm_link">
-		  <visual>
-		    <origin rpy="1.571 0 1.571" xyz="0 0 0"/>
-		    <geometry>
-		      <mesh filename="package://lift-arm-description/models/meshes/collada_files/sec_arm.dae"/>
-		    </geometry>
-		  </visual>
-		  <collision>
-		  	<origin rpy="1.571 0 1.571" xyz="0 0 0"/>
-		    <geometry>
-		      <mesh filename="package://lift-arm-description/models/meshes/collada_files/sec_arm.dae"/>
-		  	</geometry>
-		  </collision>
+			<inertial>
+				<origin rpy="0 0 0" xyz="0.021 0.000 0.009"/>
+				<mass value="0.041"/>
+				<inertia
+					ixx="0.000005"
+					ixy="-0.000000"	iyy="0.000039"
+					ixz="0.000001"	iyz="-0.000000"	izz="0.000042"
+				/>
+			</inertial>
+			<visual>
+				<origin rpy="1.571 0 1.571" xyz="0 0 0"/>
+				<geometry>
+					<mesh filename="package://lift-arm-description/models/meshes/collada_files/sec_arm.dae"/>
+				</geometry>
+			</visual>
+			<collision>
+				<origin rpy="1.571 0 1.571" xyz="0 0 0"/>
+				<geometry>
+					<mesh filename="package://lift-arm-description/models/meshes/collada_files/sec_arm.dae"/>
+				</geometry>
+				<contact_coefficients mu="1" kp="100000" kd="100000"/>
+			</collision>
 		</link>
 		<joint name="${prefix}sec_arm_joint" type="revolute">
-		  <parent link="${prefix}base_link"/>
-		  <child link="${prefix}sec_arm_link"/>
-		  <origin xyz="0 0.0095 0.044953" rpy="0 0 1.571"/>
-		  <limit lower="-0.436" upper="2.531" effort="2.236" velocity="7.480"/>
-		  <axis xyz="1 0 0"/>
-		</joint>
-		<link name="${prefix}strut_link">
-		  <visual>
-		    <origin rpy="1.571 0 1.571" xyz="0 0 0"/>
-		    <geometry>
-		      <mesh filename="package://lift-arm-description/models/meshes/collada_files/strut.dae"/>
-		    </geometry>
-		  </visual>
-		  <collision>
-		  	<origin rpy="1.571 0 1.571" xyz="0 0 0"/>
-		  	<geometry>
-		  		<mesh filename="package://lift-arm-description/models/meshes/collada_files/strut.dae"/>
-		  	</geometry>
-		  </collision>
+			<parent link="${prefix}base_link"/>
+			<child link="${prefix}sec_arm_link"/>
+			<origin xyz="0 0.0095 0.044953" rpy="0 0 1.571"/>
+			<limit lower="-0.436" upper="2.531" effort="2.236" velocity="7.480"/>
+			<axis xyz="1 0 0"/>
+		</joint>
+		<link name="${prefix}strut_link">">
+			<inertial>
+				<origin rpy="0 0 0" xyz="0.080 0 0.003"/>
+				<mass value="0.007"/>
+				<inertia
+					ixx="0.000048"
+					ixy="-0.00000"	iyy="0.000018"
+					ixz="0.00000"	iyz="-0.00000"	izz="0.000018"
+				/>
+			</inertial>
+			<visual>
+				<origin rpy="1.571 0 1.571" xyz="0 0 0"/>
+				<geometry>
+					<mesh filename="package://lift-arm-description/models/meshes/collada_files/strut.dae"/>
+				</geometry>
+			</visual>
+			<collision>
+				<origin rpy="1.571 0 1.571" xyz="0 0 0"/>
+				<geometry>
+					<mesh filename="package://lift-arm-description/models/meshes/collada_files/strut.dae"/>
+				</geometry>
+				<contact_coefficients mu="1" kp="100000" kd="100000"/>
+			</collision>
 		</link>
 		<joint name="${prefix}strut_joint_lower" type="continuous">
-		  <parent link="${prefix}sec_arm_link"/>
-		  <child link="${prefix}strut_link"/>
-		  <origin xyz="0.006 0.09 0" rpy="0 0 0"/>
-		  <axis xyz="1 0 0"/>
+			<parent link="${prefix}sec_arm_link"/>
+			<child link="${prefix}strut_link"/>
+			<origin xyz="0.006 0.09 0" rpy="0 0 0"/>
+			<axis xyz="1 0 0"/>
 		</joint>
 		<link name="${prefix}upper_arm_link">
-		  <visual>
-		    <origin rpy="1.571 0 1.571" xyz="0 0 0"/>
-		    <geometry>
-		      <mesh filename="package://lift-arm-description/models/meshes/collada_files/upper_arm.dae"/>
-		    </geometry>
-		  </visual>
-		  <collision>
-		  	<origin rpy="1.571 0 1.571" xyz="0 0 0"/>
-		  	<geometry>
-		  		<mesh filename="package://lift-arm-description/models/meshes/collada_files/upper_arm.dae"/>
-		  	</geometry>
-		  </collision>
+			<inertial>
+				<origin rpy="0 0 0" xyz="-0.081 0.024 -0.006"/>
+				<mass value="0.112"/>
+				<inertia
+					ixx="0.000036"
+					ixy="0.000055"	iyy="0.000624"
+					ixz="-0.000063"	iyz="0.000007"	izz="0.000614"
+				/>
+			</inertial>
+			<visual>
+				<origin rpy="1.571 0 1.571" xyz="0 0 0"/>
+				<geometry>
+					<mesh filename="package://lift-arm-description/models/meshes/collada_files/upper_arm.dae"/>
+				</geometry>
+			</visual>
+			<collision>
+				<origin rpy="1.571 0 1.571" xyz="0 0 0"/>
+				<geometry>
+					<mesh filename="package://lift-arm-description/models/meshes/collada_files/upper_arm.dae"/>
+				</geometry>
+				<contact_coefficients mu="1" kp="100000" kd="100000"/>
+			</collision>
 		</link>
 		<joint name="${prefix}upper_arm_joint" type="revolute">
-		  <parent link="${prefix}main_arm_link"/>
-		  <child link="${prefix}upper_arm_link"/>
-		  <origin xyz="0.0095 0 0.18" rpy="0 0 0"/>
-		  <limit lower="-0.873" upper="1.484" effort="2.236" velocity="7.480"/>
-		  <axis xyz="1 0 0"/>
+			<parent link="${prefix}main_arm_link"/>
+			<child link="${prefix}upper_arm_link"/>
+			<origin xyz="0.0095 0 0.18" rpy="0 0 0"/>
+			<limit lower="-0.873" upper="1.484" effort="2.236" velocity="7.480"/>
+			<axis xyz="1 0 0"/>
 		</joint>
 		<link name="${prefix}rack_link">
-		  <visual>
-		    <origin rpy="1.571 0 0" xyz="0 0 0"/>
-		    <geometry>
-		      <mesh filename="package://lift-arm-description/models/meshes/collada_files/rack.dae"/>
-		    </geometry>
-		  </visual>
-		  <collision>
-		  	<origin rpy="1.571 0 0" xyz="0 0 0"/>
-		  	<geometry>
-		  		<mesh filename="package://lift-arm-description/models/meshes/collada_files/rack.dae"/>
-		  	</geometry>
-		  </collision>
+			<inertial>
+				<origin rpy="0 0 0" xyz="0.130 0.001 0.000"/>
+				<mass value="0.026"/>
+				<inertia
+					ixx="0.000000"
+					ixy="-0.000001"	iyy="0.000241"
+					ixz="0.000000"	iyz="0.000000"	izz="0.000241"
+				/>
+			</inertial>
+			<visual>
+				<origin rpy="1.571 0 0" xyz="0 0 0"/>
+				<geometry>
+					<mesh filename="package://lift-arm-description/models/meshes/collada_files/rack.dae"/>
+				</geometry>
+			</visual>
+			<collision>
+				<origin rpy="1.571 0 0" xyz="0 0 0"/>
+				<geometry>
+					<mesh filename="package://lift-arm-description/models/meshes/collada_files/rack.dae"/>
+				</geometry>
+				<contact_coefficients mu="1" kp="100000" kd="100000"/>
+			</collision>
 		</link>
 		<joint name="${prefix}rack_joint" type="prismatic">
@@ -124,6 +184,36 @@
 			<parent link="${prefix}rack_link"/>
 			<child link="${prefix}end_effector_link"/>
-			<origin xyz="0 0 0.033" rpy="0 0 0"/>
-		</joint>
+			<origin xyz="0.02 0 0" rpy="0 0 0"/>
+		</joint>
+		<transmission name="tran1">
+			<type>transmission_interface/SimpleTransmission</type>
+			<joint name="main_arm_joint">
+				<hardwareInterface>EffortJointInterface</hardwareInterface>
+			</joint>
+			<actuator name="servo1">
+				<hardwareInterface>EffortJointInterface</hardwareInterface>
+				<mechanicalReduction>1</mechanicalReduction>
+			</actuator>
+		</transmission>
+		<transmission name="tran2">
+			<type>transmission_interface/SimpleTransmission</type>
+			<joint name="upper_arm_joint">
+				<hardwareInterface>EffortJointInterface</hardwareInterface>
+			</joint>
+			<actuator name="servo2">
+				<hardwareInterface>EffortJointInterface</hardwareInterface>
+				<mechanicalReduction>1</mechanicalReduction>
+			</actuator>
+		</transmission>
+		<transmission name="tran3">
+			<type>transmission_interface/SimpleTransmission</type>
+			<joint name="rack_joint">
+				<hardwareInterface>EffortJointInterface</hardwareInterface>
+			</joint>
+			<actuator name="stepper">
+				<hardwareInterface>EffortJointInterface</hardwareInterface>
+				<mechanicalReduction>1</mechanicalReduction>
+			</actuator>
+		</transmission>
 	</xacro:macro>
 </robot>

Commit message: small model fix

File: robot/manipulator_macro.xacro (robot description, xacro)
@@ -160,5 +160,5 @@
 			</inertial>
 			<visual>
-				<origin rpy="1.571 0 0" xyz="0 0 0"/>
+				<origin rpy="1.571 0 3.1415" xyz="0 0 0"/>
 				<geometry>
 					<mesh filename="package://lift-arm-description/models/meshes/collada_files/rack.dae"/>
@@ -166,5 +166,5 @@
 			</visual>
 			<collision>
-				<origin rpy="1.571 0 0" xyz="0 0 0"/>
+				<origin rpy="1.571 0 3.1415" xyz="0 0 0"/>
 				<geometry>
 					<mesh filename="package://lift-arm-description/models/meshes/collada_files/rack.dae"/>
@@ -176,5 +176,5 @@
 			<parent link="${prefix}upper_arm_link"/>
 			<child link="${prefix}rack_link"/>
-			<origin xyz="0 0 0.033" rpy="0 0 -1.571"/>
+			<origin xyz="0 -0.30 0.033" rpy="0 0 -1.571"/>
 			<limit lower="-0.1" upper="0.15" effort="3.43" velocity="0.0314"/>
 			<axis xyz="1 0 0"/>

Commit message: name change, gazebo integration

File: robot/manipulator_macro.xacro (robot description, xacro)
@@ -1,5 +1,5 @@
 <?xml version="1.0"?>
 <robot xmlns:xacro="http://ros.org/wiki/xacro">
-	<xacro:macro name="lift-arm" params="prefix">
+	<xacro:macro name="lift_arm" params="prefix">
 		<link name="${prefix}base_link">
 			<inertial>
@@ -15,5 +15,5 @@
 				<origin rpy="0 0 3.142" xyz="0 0 0"/>
 				<geometry>
-					<mesh filename="package://lift-arm-description/models/meshes/collada_files/base.dae"/>
+					<mesh filename="package://lift_arm_description/models/meshes/collada_files/base.dae"/>
 				</geometry>
 			</visual>
@@ -21,5 +21,5 @@
 				<origin rpy="0 0 3.142" xyz="0 0 0"/>
 				<geometry>
-					<mesh filename="package://lift-arm-description/models/meshes/collada_files/base.dae"/>
+					<mesh filename="package://lift_arm_description/models/meshes/collada_files/base.dae"/>
 				</geometry>
 				<contact_coefficients mu="1" kp="100000" kd="100000"/>
@@ -39,5 +39,5 @@
 				<origin rpy="1.571 -1.571 1.571" xyz="0 0 0"/>
 				<geometry>
-					<mesh filename="package://lift-arm-description/models/meshes/collada_files/main_arm.dae"/>
+					<mesh filename="package://lift_arm_description/models/meshes/collada_files/main_arm.dae"/>
 				</geometry>
 			</visual>
@@ -45,5 +45,5 @@
 				<origin rpy="1.571 -1.571 1.571" xyz="0 0 0"/>
 				<geometry>
-					<mesh filename="package://lift-arm-description/models/meshes/collada_files/main_arm.dae"/>
+					<mesh filename="package://lift_arm_description/models/meshes/collada_files/main_arm.dae"/>
 				</geometry>
 				<contact_coefficients mu="1" kp="100000" kd="100000"/>
@@ -56,4 +56,5 @@
 			<limit lower="-1.920" upper="1.134" effort="2.236" velocity="7.480"/>
 			<axis xyz="1 0 0"/>
+			<dynamics damping="0.7"/>
 		</joint>
 		<link name="${prefix}sec_arm_link">
@@ -70,11 +71,11 @@
 				<origin rpy="1.571 0 1.571" xyz="0 0 0"/>
 				<geometry>
-					<mesh filename="package://lift-arm-description/models/meshes/collada_files/sec_arm.dae"/>
-				</geometry>
-			</visual>
-			<collision>
-				<origin rpy="1.571 0 1.571" xyz="0 0 0"/>
-				<geometry>
-					<mesh filename="package://lift-arm-description/models/meshes/collada_files/sec_arm.dae"/>
+					<mesh filename="package://lift_arm_description/models/meshes/collada_files/sec_arm.dae"/>
+				</geometry>
+			</visual>
+			<collision>
+				<origin rpy="1.571 0 1.571" xyz="0 0 0"/>
+				<geometry>
+					<mesh filename="package://lift_arm_description/models/meshes/collada_files/sec_arm.dae"/>
 				</geometry>
 				<contact_coefficients mu="1" kp="100000" kd="100000"/>
@@ -87,4 +88,5 @@
 			<limit lower="-0.436" upper="2.531" effort="2.236" velocity="7.480"/>
 			<axis xyz="1 0 0"/>
+			<dynamics damping="0.7"/>
 		</joint>
 		<link name="${prefix}strut_link">">
@@ -101,11 +103,11 @@
 				<origin rpy="1.571 0 1.571" xyz="0 0 0"/>
 				<geometry>
-					<mesh filename="package://lift-arm-description/models/meshes/collada_files/strut.dae"/>
-				</geometry>
-			</visual>
-			<collision>
-				<origin rpy="1.571 0 1.571" xyz="0 0 0"/>
-				<geometry>
-					<mesh filename="package://lift-arm-description/models/meshes/collada_files/strut.dae"/>
+					<mesh filename="package://lift_arm_description/models/meshes/collada_files/strut.dae"/>
+				</geometry>
+			</visual>
+			<collision>
+				<origin rpy="1.571 0 1.571" xyz="0 0 0"/>
+				<geometry>
+					<mesh filename="package://lift_arm_description/models/meshes/collada_files/strut.dae"/>
 				</geometry>
 				<contact_coefficients mu="1" kp="100000" kd="100000"/>
@@ -131,11 +133,11 @@
 				<origin rpy="1.571 0 1.571" xyz="0 0 0"/>
 				<geometry>
-					<mesh filename="package://lift-arm-description/models/meshes/collada_files/upper_arm.dae"/>
-				</geometry>
-			</visual>
-			<collision>
-				<origin rpy="1.571 0 1.571" xyz="0 0 0"/>
-				<geometry>
-					<mesh filename="package://lift-arm-description/models/meshes/collada_files/upper_arm.dae"/>
+					<mesh filename="package://lift_arm_description/models/meshes/collada_files/upper_arm.dae"/>
+				</geometry>
+			</visual>
+			<collision>
+				<origin rpy="1.571 0 1.571" xyz="0 0 0"/>
+				<geometry>
+					<mesh filename="package://lift_arm_description/models/meshes/collada_files/upper_arm.dae"/>
 				</geometry>
 				<contact_coefficients mu="1" kp="100000" kd="100000"/>
@@ -148,4 +150,5 @@
 			<limit lower="-0.873" upper="1.484" effort="2.236" velocity="7.480"/>
 			<axis xyz="1 0 0"/>
+			<dynamics damping="0.7"/>
 		</joint>
 		<link name="${prefix}rack_link">
@@ -162,5 +165,5 @@
 				<origin rpy="1.571 0 3.1415" xyz="0 0 0"/>
 				<geometry>
-					<mesh filename="package://lift-arm-description/models/meshes/collada_files/rack.dae"/>
+					<mesh filename="package://lift_arm_description/models/meshes/collada_files/rack.dae"/>
 				</geometry>
 			</visual>
@@ -168,5 +171,5 @@
 				<origin rpy="1.571 0 3.1415" xyz="0 0 0"/>
 				<geometry>
-					<mesh filename="package://lift-arm-description/models/meshes/collada_files/rack.dae"/>
+					<mesh filename="package://lift_arm_description/models/meshes/collada_files/rack.dae"/>
 				</geometry>
 				<contact_coefficients mu="1" kp="100000" kd="100000"/>
@@ -186,30 +189,30 @@
 			<origin xyz="0.02 0 0" rpy="0 0 0"/>
 		</joint>
-		<transmission name="tran1">
+		<transmission name="${prefix}tran1">
 			<type>transmission_interface/SimpleTransmission</type>
-			<joint name="main_arm_joint">
+			<joint name="${prefix}main_arm_joint">
 				<hardwareInterface>EffortJointInterface</hardwareInterface>
 			</joint>
-			<actuator name="servo1">
+			<actuator name="${prefix}servo1">
 				<hardwareInterface>EffortJointInterface</hardwareInterface>
 				<mechanicalReduction>1</mechanicalReduction>
 			</actuator>
 		</transmission>
-		<transmission name="tran2">
+		<transmission name="${prefix}tran2">
 			<type>transmission_interface/SimpleTransmission</type>
-			<joint name="upper_arm_joint">
+			<joint name="${prefix}upper_arm_joint">
 				<hardwareInterface>EffortJointInterface</hardwareInterface>
 			</joint>
-			<actuator name="servo2">
+			<actuator name="${prefix}servo2">
 				<hardwareInterface>EffortJointInterface</hardwareInterface>
 				<mechanicalReduction>1</mechanicalReduction>
 			</actuator>
 		</transmission>
-		<transmission name="tran3">
+		<transmission name="${prefix}tran3">
 			<type>transmission_interface/SimpleTransmission</type>
-			<joint name="rack_joint">
+			<joint name="${prefix}rack_joint">
 				<hardwareInterface>EffortJointInterface</hardwareInterface>
 			</joint>
-			<actuator name="stepper">
+			<actuator name="${prefix}stepper">
 				<hardwareInterface>EffortJointInterface</hardwareInterface>
 				<mechanicalReduction>1</mechanicalReduction>

File: urdf/manipulator.urdf (robot description, URDF)
Before this commit: robot lift-arm, 6 links, 5 joints
Links:
- added link end_effector_link
- link base_link: mass None -> 0.873
- link main_arm_link: mass None -> 0.108
- link rack_link: mass None -> 0.026
- link sec_arm_link: mass None -> 0.041
- link strut_link: mass None -> 0.007
- link upper_arm_link: mass None -> 0.112
Joints:
- added joint enef_joint: type fixed, parent rack_link, child end_effector_link, origin xyz=0.02 0 0 rpy=0 0 0
- joint main_arm_joint: limit lower=-1.920 upper=1.134 effort=0.1 velocity=0.005 -> lower=-1.920 upper=1.134 effort=2.236 velocity=7.480
- joint rack_joint: limit lower=-0.1 upper=0.15 effort=0.1 velocity=0.005 -> lower=-0.1 upper=0.15 effort=3.43 velocity=0.0314; origin xyz=0 0 0.033 rpy=0 0 -1.571 -> xyz=0 -0.30 0.033 rpy=0 0 -1.571
- joint sec_arm_joint: limit lower=-0.436 upper=2.531 effort=0.1 velocity=0.005 -> lower=-0.436 upper=2.531 effort=2.236 velocity=7.480
- joint upper_arm_joint: limit lower=-0.873 upper=1.484 effort=0.1 velocity=0.005 -> lower=-0.873 upper=1.484 effort=2.236 velocity=7.480

Commit message: Update manipulator_macro.xacro

File: robot/manipulator_macro.xacro (robot description, xacro)
@@ -54,5 +54,5 @@
 			<child link="${prefix}main_arm_link"/>
 			<origin xyz="0 -0.0095 0.044953" rpy="0 0 1.571"/>
-			<limit lower="-1.920" upper="1.134" effort="2.236" velocity="7.480"/>
+			<limit lower="-1.658" upper="1.047" effort="2.236" velocity="7.480"/>
 			<axis xyz="1 0 0"/>
 			<dynamics damping="0.7"/>
@@ -86,5 +86,5 @@
 			<child link="${prefix}sec_arm_link"/>
 			<origin xyz="0 0.0095 0.044953" rpy="0 0 1.571"/>
-			<limit lower="-0.436" upper="2.531" effort="2.236" velocity="7.480"/>
+			<limit lower="-0.436" upper="2.601" effort="2.236" velocity="7.480"/>
 			<axis xyz="1 0 0"/>
 			<dynamics damping="0.7"/>
